Commit message: Updated the Ackermann steering

File: trackday/urdf/racecar.urdf (robot description, URDF)
Before this commit: robot racecar, 8 links, 7 joints
Joints:
- joint front_left_steering_joint: limit lower=-0.6 upper=0.6 effort=50 velocity=1.0 -> lower=-0.6 upper=0.6 effort=50 velocity=10
- joint front_right_steering_joint: limit lower=-0.6 upper=0.6 effort=50 velocity=1.0 -> lower=-0.6 upper=0.6 effort=50 velocity=10

Commit message: Adjusted the scaling

File: trackday/urdf/racecar.urdf (robot description, URDF)
Before this commit: robot racecar, 8 links, 7 joints
Links:
- link base_link: mass 15.0 -> 150.0; geometry collision mesh filename=package://trackday/meshes/car.stl scale=0.1 0.1 0.1; visual mesh filename=package://trackday/meshes/car.dae scale=0.1 0.1 0.1
- link front_left_steering_link: mass 0.5 -> 0.3
- link front_left_wheel: mass 5.0 -> 1.5; geometry collision mesh filename=package://trackday/meshes/rim.dae scale=0.1 0.1 0.1; visual mesh filename=package://trackday/meshes/rim.dae scale=0.1 0.1 0.1
- link front_right_steering_link: mass 0.5 -> 0.3
- link front_right_wheel: mass 5.0 -> 1.5; geometry collision mesh filename=package://trackday/meshes/rim.dae scale=0.1 0.1 0.1; visual mesh filename=package://trackday/meshes/rim.dae scale=0.1 0.1 0.1
- link rear_left_wheel: mass 5.0 -> 1.5; geometry collision mesh filename=package://trackday/meshes/rim.dae scale=0.1 0.1 0.1; visual mesh filename=package://trackday/meshes/rim.dae scale=0.1 0.1 0.1
- link rear_right_wheel: mass 5.0 -> 1.5; geometry collision mesh filename=package://trackday/meshes/rim.dae scale=0.1 0.1 0.1; visual mesh filename=package://trackday/meshes/rim.dae scale=0.1 0.1 0.1
Joints:
- joint base_footprint_joint: origin xyz=0 0 0 rpy=0 0 0 -> xyz=0 0 0 rpy=0 0 1.5707
- joint front_left_steering_joint: limit lower=-0.6 upper=0.6 effort=50 velocity=10 -> lower=-0.6 upper=0.6 effort=1000 velocity=10; origin xyz=1.5 -1.8 -0.7 rpy=0 0 0 -> xyz=0.15 -0.18 -0.07 rpy=0 0 0
- joint front_right_steering_joint: limit lower=-0.6 upper=0.6 effort=50 velocity=10 -> lower=-0.6 upper=0.6 effort=1000 velocity=10; origin xyz=-1.5 -1.8 -0.7 rpy=0 0 0 -> xyz=-0.15 -0.18 -0.07 rpy=0 0 0
- joint rear_left_wheel_joint: limit effort=100 velocity=10 -> effort=1000 velocity=10; origin xyz=1.5 3.1 -0.7 rpy=0 0 0 -> xyz=0.15 0.31 -0.07 rpy=0 0 0
- joint rear_right_wheel_joint: limit effort=100 velocity=10 -> effort=1000 velocity=10; origin xyz=-1.5 3.1 -0.7 rpy=0 0 0 -> xyz=-0.15 0.31 -0.07 rpy=0 0 0

Commit message: Updated wheel collision

File: trackday/urdf/racecar.urdf (robot description, URDF)
Before this commit: robot racecar, 8 links, 7 joints
Links:
- link front_left_wheel: geometry collision cylinder length=.05 radius=0.072; visual mesh filename=package://trackday/meshes/rim.dae scale=0.1 0.1 0.1
- link front_right_wheel: geometry collision cylinder length=.05 radius=0.072; visual mesh filename=package://trackday/meshes/rim.dae scale=0.1 0.1 0.1
- link rear_left_wheel: geometry collision cylinder length=.05 radius=0.072; visual mesh filename=package://trackday/meshes/rim.dae scale=0.1 0.1 0.1
- link rear_right_wheel: geometry collision cylinder length=.05 radius=0.072; visual mesh filename=package://trackday/meshes/rim.dae scale=0.1 0.1 0.1

Commit message: Fixed model axis

File: trackday/urdf/racecar.urdf (robot description, URDF)
Before this commit: robot racecar, 8 links, 7 joints
Joints:
- joint base_footprint_joint: origin xyz=0 0 0 rpy=0 0 1.5707 -> xyz=0 0 0 rpy=0 0 0
- joint front_left_steering_joint: origin xyz=0.15 -0.18 -0.07 rpy=0 0 0 -> xyz=0.18 0.15 -0.07 rpy=0 0 0
- joint front_left_wheel_joint: axis 1 0 0 -> 0 1 0
- joint front_right_steering_joint: origin xyz=-0.15 -0.18 -0.07 rpy=0 0 0 -> xyz=0.18 -0.15 -0.07 rpy=0 0 0
- joint front_right_wheel_joint: axis 1 0 0 -> 0 1 0
- joint rear_left_wheel_joint: axis 1 0 0 -> 0 1 0; origin xyz=0.15 0.31 -0.07 rpy=0 0 0 -> xyz=-0.31 0.15 -0.07 rpy=0 0 0
- joint rear_right_wheel_joint: axis 1 0 0 -> 0 1 0; origin xyz=-0.15 0.31 -0.07 rpy=0 0 0 -> xyz=-0.31 -0.15 -0.07 rpy=0 0 0

Commit message: Added camera to the robot

File: trackday/urdf/racecar.urdf (robot description, URDF)
Before this commit: robot racecar, 8 links, 7 joints
Links:
- added link camera_link, mass 0.1; collision box size=.03 .03 .03; visual box size=.03 .03 .03
- added link camera_link_optical
Joints:
- added joint camera_joint: type fixed, parent base_link, child camera_link, origin xyz=-0.015 0 0.2 rpy=0 0 0, axis 0 1 0
- added joint camera_optical_joint: type fixed, parent camera_link, child camera_link_optical, origin xyz=0 0 0 rpy=-1.5707 0 -1.5707

Commit message: Fixed OpenCV

File: trackday/urdf/racecar.urdf (robot description, URDF)
Before this commit: robot racecar, 10 links, 9 joints
Links:
- link base_link: geometry collision mesh filename=package://trackday/meshes/car.dae scale=0.1 0.1 0.1; visual mesh filename=package://trackday/meshes/car.dae scale=0.1 0.1 0.1
Joints:
- joint camera_joint: origin xyz=-0.015 0 0.2 rpy=0 0 0 -> xyz=0.32 0 0.1 rpy=0 0.414 0
- joint front_left_steering_joint: limit lower=-0.6 upper=0.6 effort=1000 velocity=10 -> lower=-0.6 upper=0.6 effort=100000 velocity=10
- joint front_right_steering_joint: limit lower=-0.6 upper=0.6 effort=1000 velocity=10 -> lower=-0.6 upper=0.6 effort=100000 velocity=10
